File: universal_board/universal_board_manu/universal_board.kicad_pcb (KiCad board)
At the start: 2 copper layers, 83.3 x 92.5 mm, 54 parts

Commit message: board
Parts:
- removed 19 (x2), 20 (x2), 21 (x2), 22 (x2), 23 (x2), 24 (x2), 25 (x2), 26 (x2), 27 (x2): , 
- removed the ? at (150.0, 77.2)
- removed the ? at (192.8, 124.0)
- added REF**: PinSocket_1x10_P2.54mm_Vertical, Connector_PinSocket_2.54mm:PinSocket_1x10_P2.54mm_Vertical, F.Cu at (139.1, 124.2)
- added REF**: PinSocket_1x10_P2.54mm_Vertical, Connector_PinSocket_2.54mm:PinSocket_1x10_P2.54mm_Vertical, F.Cu at (195.0, 123.8)
- added REF**: JST_GH_SM02B-GHS-TB_1x02-1MP_P1.25mm_Horizontal, Connector_JST:JST_GH_SM02B-GHS-TB_1x02-1MP_P1.25mm_Horizontal, F.Cu at (152.1, 117.1)
- moved dawdad 58.2 mm to (161.0, 108.4)
- moved dadada 48.7 mm to (160.8, 86.8)
- moved REF** 40.1 mm to (161.9, 98.5)
- moved 3 39.7 mm to (152.3, 101.9)
- moved 1 39.7 mm to (152.3, 106.9)
- moved 2 39.7 mm to (152.3, 104.4)
- moved 4 39.7 mm to (152.3, 99.3)
- moved 6 39.7 mm to (152.3, 94.2)
- moved 8 39.7 mm to (165.8, 104.6)
- moved ? 39.7 mm to (152.3, 109.5)
- moved 2 39.7 mm to (164.6, 104.2)
- moved 5 39.7 mm to (152.3, 96.8)
- moved 9 39.7 mm to (167.0, 104.6)
- moved ? 39.7 mm to (164.5, 104.6)
- moved 7 39.7 mm to (164.6, 100.7)
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Connections:
- 18 pad : 5V -> 3.3V
Routing:
- net GND: track 187.7 -> 0.00 mm, vias 3 -> 0
- net 5V: track 161.9 -> 0.00 mm, vias 2 -> 0
- net 14: track 105.9 -> 0.00 mm, vias 3 -> 0
- net 4: track 94.7 -> 0.00 mm, vias 2 -> 0
- net 15: track 94.6 -> 0.00 mm, vias 4 -> 0
- net IR: track 90.9 -> 0.00 mm
- net 3.3V: track 84.5 -> 0.00 mm, vias 2 -> 0
- net 13: track 74.2 -> 0.00 mm, vias 4 -> 0
- net 5: track 65.5 -> 0.00 mm, vias 1 -> 0
- net 6: track 57.3 -> 0.00 mm, vias 1 -> 0
- net R_LED: track 55.6 -> 0.00 mm
- net 7: track 26.9 -> 0.00 mm, vias 2 -> 0
- net 3: track 26.8 -> 0.00 mm
- net 2: track 26.5 -> 0.00 mm
- net 1: track 25.5 -> 0.00 mm
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Other:
- board size 83.3 x 92.5 mm -> 100.9 x 55.5 mm

Commit message: kari
Parts:
- moved 9 147.8 mm to (27.4, 56.3), turned to 180 degrees
- moved 8 145.4 mm to (28.6, 56.3), turned to 180 degrees
- moved ? 143.0 mm to (29.9, 56.3), turned to 180 degrees
- moved 2 140.1 mm to (33.7, 54.5), turned to -90 degrees
- moved 7 137.7 mm to (33.7, 58.0), turned to -90 degrees
- moved dawdad 136.6 mm to (37.3, 50.2), turned to 0 degrees
- moved REF** 130.8 mm to (36.6, 61.1), turned to 180 degrees
- moved REF** 130.1 mm to (46.2, 41.5), turned to -90 degrees
- moved dadada 124.3 mm to (37.5, 71.9), turned to 0 degrees
- moved ? 122.2 mm to (46.0, 49.2), turned to -90 degrees
- moved REF** 120.2 mm to (59.2, 34.4), turned to -90 degrees
- moved 1 119.8 mm to (46.0, 51.7), turned to -90 degrees
- moved 2 117.6 mm to (46.0, 54.2), turned to -90 degrees
- moved 17 115.9 mm to (109.2, 38.0)
- moved ? 115.9 mm to (106.7, 38.0)
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Routing:
- net GND: track 0.00 -> 184.8 mm, vias 0 -> 2
- net 5V: track 0.00 -> 153.8 mm, vias 0 -> 3
- net 14: track 0.00 -> 120.4 mm, vias 0 -> 3
- net 3.3V: track 0.00 -> 119.1 mm
- net 15: track 0.00 -> 103.4 mm, vias 0 -> 4
- net 4: track 0.00 -> 102.2 mm
- net IR: track 0.00 -> 90.8 mm
- net 13: track 0.00 -> 74.3 mm, vias 0 -> 1
- net 5: track 0.00 -> 66.1 mm, vias 0 -> 2
- net 6: track 0.00 -> 65.8 mm, vias 0 -> 2
- net 7: track 0.00 -> 52.3 mm, vias 0 -> 1
- net R_LED: track 0.00 -> 45.1 mm
- net 8: track 0.00 -> 26.3 mm, vias 0 -> 2
- net 3: track 0.00 -> 25.0 mm, vias 0 -> 1
- net 1: track 0.00 -> 23.4 mm, vias 0 -> 2
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Other:
- board size 100.9 x 55.5 mm -> 95.8 x 56.2 mm

Commit message: board2
Parts:
- moved ? 110.5 mm to (128.6, 106.1)
- moved REF** 110.5 mm to (148.9, 126.7)
- moved REF** 110.5 mm to (157.9, 84.1)
- moved dawdad 110.5 mm to (136.0, 100.0)
- moved 1 110.5 mm to (144.7, 101.4)
- moved 2 110.5 mm to (144.7, 104.0)
- moved 2 110.5 mm to (132.3, 104.2)
- moved 3 110.5 mm to (144.7, 106.5)
- moved 4 110.5 mm to (144.7, 109.0)
- moved 5 110.5 mm to (144.7, 111.6)
- moved 6 110.5 mm to (144.7, 114.1)
- moved 7 110.5 mm to (132.3, 107.7)
- moved 8 110.5 mm to (127.3, 106.1)
- moved 9 110.5 mm to (126.0, 106.1)
- moved ? 110.5 mm to (144.7, 98.9)
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Other:
- board size 95.8 x 56.2 mm -> 92.8 x 103.5 mm

Commit message: new design
Parts:
- moved 2 47.7 mm to (146.0, 56.2)
- moved 4 47.7 mm to (146.0, 61.3)
- moved 8 47.7 mm to (128.7, 58.3)
- moved 9 47.7 mm to (127.4, 58.3)
- moved ? 47.7 mm to (129.9, 58.3)
- moved ? 47.7 mm to (146.0, 51.2)
- moved REF** 47.7 mm to (159.2, 36.4)
- moved REF** 47.7 mm to (136.6, 63.1)
- moved 1 47.7 mm to (146.0, 53.7)
- moved 2 47.7 mm to (133.7, 56.5)
- moved 3 47.7 mm to (146.0, 58.8)
- moved 5 47.7 mm to (146.0, 63.9)
- moved 6 47.7 mm to (146.0, 66.4)
- moved 7 47.7 mm to (133.7, 60.0)
- moved REF** 47.7 mm to (150.2, 79.0)
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Other:
- board size 92.8 x 103.5 mm -> 94.2 x 55.7 mm
