File: universal_board/universal_board_bottom/universal_board.kicad_pcb (KiCad board)
At the start: 2 copper layers, 83.3 x 92.5 mm, 54 parts

Commit message: case and MQTT
Parts:
- removed 10, 11, 12, 13, 14, 15, 16, 17, 18: , 
- removed the 19 at (195.4, 124.0)
- removed the 19 at (152.5, 77.2)
- removed the 2 at (162.8, 66.1)
- removed the 2 at (175.1, 65.9)
- removed the 20 at (197.9, 124.0)
- removed the 20 at (155.1, 77.2)
- removed the 21 at (157.6, 77.2)
- removed the 21 at (200.4, 124.0)
- removed the 22 at (203.0, 124.0)
- removed the 22 at (160.2, 77.2)
- removed the 23 at (205.5, 124.0)
- removed the 23 at (162.7, 77.2)
- removed the 24 at (165.2, 77.2)
- removed the 24 at (208.1, 124.0)
- removed the 25 at (210.6, 124.0)
- removed the 25 at (167.8, 77.2)
- removed the 26 at (213.1, 124.0)
- removed the 26 at (170.3, 77.2)
- removed the 27 at (215.7, 124.0)
- removed the 27 at (172.9, 77.2)
- removed the ? at (199.0, 72.8)
- removed the ? at (208.3, 72.3)
- removed the ? at (175.0, 66.3)
- removed the ? at (150.0, 77.2)
- removed the ? at (192.8, 124.0)
- removed the ? at (202.9, 108.5)
- removed the ? at (189.3, 72.7)
- removed the ? at (219.2, 72.3)
- removed the ? at (162.8, 71.2)
- removed the ? at (191.9, 72.7)
- removed the REF** at (191.5, 119.8)
- removed the REF** at (196.7, 114.0)
- removed the REF** at (203.3, 112.2)
- removed the REF** at (173.2, 60.0)
- added 19: , , F.Cu at (217.9, 71.8)
- added 2: , , F.Cu at (228.2, 60.6)
- added 2: , , F.Cu at (240.5, 60.4)
- added 20: , , F.Cu at (220.5, 71.8)
- added 21: , , F.Cu at (223.0, 71.8)
- added 22: , , F.Cu at (225.6, 71.8)
- added 23: , , F.Cu at (228.1, 71.8)
- added 24: , , F.Cu at (230.7, 71.8)
- added 25: , , F.Cu at (233.2, 71.8)
- added 26: , , F.Cu at (235.7, 71.8)
- added 27: , , F.Cu at (238.3, 71.8)
- added ?: , , F.Cu at (240.4, 60.9)
- added ?: , , F.Cu at (215.4, 71.8)
- added ?: , , F.Cu at (228.2, 65.7)
- added REF**: R_Axial_DIN0204_L3.6mm_D1.6mm_P5.08mm_Horizontal, Resistor_THT:R_Axial_DIN0204_L3.6mm_D1.6mm_P5.08mm_Horizontal, F.Cu at (238.7, 54.5)
- moved 1 65.6 mm to (228.2, 63.2)
- moved 3 65.6 mm to (228.2, 58.1)
- moved 4 65.6 mm to (228.2, 55.5)
- moved 5 65.6 mm to (228.2, 53.0)
- moved 6 65.6 mm to (228.2, 50.5)
- moved 7 65.6 mm to (240.5, 56.9)
- moved 8 65.6 mm to (241.7, 60.9)
- moved 9 65.6 mm to (242.9, 60.9)
- moved REF** 65.6 mm to (224.0, 37.9)
- moved dadada 65.6 mm to (237.0, 33.8)
- moved dawdad 65.6 mm to (237.1, 45.7)
Routing:
- net GND: track 187.7 -> 97.1 mm, vias 3 -> 2
- net 5V: track 161.9 -> 72.2 mm, vias 2 -> 0
- net IR: track 90.9 -> 23.7 mm
- net 14: track 105.9 -> 45.6 mm, vias 3 -> 1
- net R_LED: track 55.6 -> 0.00 mm
- net 4: track 94.7 -> 40.0 mm
- net 15: track 94.6 -> 42.9 mm
- net 3.3V: track 84.5 -> 44.5 mm
- net 5: track 65.5 -> 41.4 mm
- net 6: track 57.3 -> 36.5 mm
- net 13: track 74.2 -> 53.5 mm, vias 4 -> 3
Other:
- board size 83.3 x 92.5 mm -> 39.1 x 45.8 mm
- board text removed: "${REFERENCE}"
- board text removed: "32Ω"
- board text removed: "47kΩ"
- board text removed: "RGBLED"
- board text removed: "光センサ"
- board text removed: "決定用タクトスイッチ"
- board text removed: "赤外線LED"
- board text removed: "赤外線センサー"

Commit message: OLED 0.1
Parts:
- removed 19, 20, 21, 22, 23, 24, 25, 26, 27: , 
- removed the 2 at (228.2, 60.6)
- removed the 2 at (240.5, 60.4)
- removed the ? at (240.4, 60.9)
- removed the ? at (215.4, 71.8)
- removed the ? at (228.2, 65.7)
- added 2: , , F.Cu at (211.4, 81.6)
- added 2: , , F.Cu at (199.1, 81.9)
- added ?: , , F.Cu at (195.3, 83.7)
- added ?: , , F.Cu at (211.4, 76.6)
- added REF**: PinSocket_1x10_P2.54mm_Vertical, Connector_PinSocket_2.54mm:PinSocket_1x10_P2.54mm_Vertical, F.Cu at (224.6, 61.8)
- added REF**: JST_GH_SM02B-GHS-TB_1x02-1MP_P1.25mm_Horizontal, Connector_JST:JST_GH_SM02B-GHS-TB_1x02-1MP_P1.25mm_Horizontal, F.Cu at (211.6, 68.9)
- moved dadada 73.9 mm to (202.9, 99.3), turned to 0 degrees
- moved REF** 67.1 mm to (215.6, 104.4), turned to 180 degrees
- moved 9 55.2 mm to (192.7, 83.7), turned to 180 degrees
- moved 8 52.9 mm to (194.0, 83.7), turned to 180 degrees
- moved 7 50.3 mm to (199.1, 85.4), turned to -90 degrees
- moved REF** 50.0 mm to (201.9, 88.5), turned to 180 degrees
- moved dawdad 46.9 mm to (202.7, 77.7), turned to 0 degrees
- moved 6 44.6 mm to (211.4, 91.8), turned to -90 degrees
- moved 5 40.0 mm to (211.4, 89.3), turned to -90 degrees
- moved 4 35.4 mm to (211.4, 86.7), turned to -90 degrees
- moved 3 31.1 mm to (211.4, 84.2), turned to -90 degrees
- moved 1 23.2 mm to (211.4, 79.1), turned to -90 degrees
Routing:
- net 7: track 26.9 -> 52.3 mm, vias 2 -> 1
- net 5V: track 72.2 -> 92.0 mm, vias 0 -> 2
- net A_GND: track 0.00 -> 18.4 mm
- net 14: track 45.6 -> 63.2 mm, vias 1 -> 3
- net IR: track 23.7 -> 40.3 mm
- net 8: track 9.90 -> 26.3 mm
- net 6: track 36.5 -> 50.7 mm, vias 1 -> 2
- net 9: track 9.37 -> 23.2 mm, vias 2 -> 1
- net A_V: track 0.00 -> 12.0 mm
- net 4: track 40.0 -> 51.7 mm, vias 2 -> 0
- net 11: track 17.0 -> 5.87 mm, vias 2 -> 1
- net 10: track 15.9 -> 6.27 mm, vias 2 -> 1
- net 5: track 41.4 -> 50.9 mm, vias 1 -> 2
- net 15: track 42.9 -> 50.4 mm, vias 4 -> 2
- net 13: track 53.5 -> 58.5 mm, vias 3 -> 1
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Other:
- board size 39.1 x 45.8 mm -> 45 x 54.9 mm
